Commit message: Up to new

File: description/lidar.xacro (robot description, xacro)
@@ -4,5 +4,5 @@
         <parent link="chassis"/>
         <child link="laser_frame"/>
-        <origin xyz="0.050 0 0.145" rpy="0 0 0"/>
+        <origin xyz="0.100 0 0.145" rpy="0 0 0"/>
     </joint>
     <link name="laser_frame">
@@ -33,5 +33,5 @@
         <sensor name="laser" type="ray">
             <pose> 0 0 0 0 0 0 </pose>
-            <visualize>false</visualize>
+            <visualize>true</visualize>
             <update_rate>10</update_rate>
             <ray>

File: description/robot.urdf.xacro (robot description, xacro)
@@ -10,4 +10,4 @@
     </xacro:unless>
     <xacro:include filename="lidar.xacro" />
-    <xacro:include filename="camera.xacro" />
+    <!--xacro:include filename="camera.xacro" />-->
 </robot>

File: description/robot_core.xacro (robot description, xacro)
@@ -9,5 +9,5 @@
     <xacro:property name="wheel_thickness" value="0.026"/>
     <xacro:property name="wheel_mass" value="0.05"/>
-    <xacro:property name="wheel_offset_x" value="0.215"/>
+    <xacro:property name="wheel_offset_x" value="0.195"/>
     <xacro:property name="wheel_offset_y" value="0.1165"/>
     <xacro:property name="wheel_offset_z" value="0.0157"/>
